Commit message: Added meshes. Added HDL-32E.

File: velodyne_description/urdf/HDL-32E.urdf.xacro (robot description, xacro)
@@ -1,5 +1,5 @@
 <?xml version="1.0"?>
-<robot xmlns:xacro="http://ros.org/wiki/xacro" name="VLP-16">
-  <xacro:macro name="VLP-16" params="parent name *origin">
+<robot xmlns:xacro="http://ros.org/wiki/xacro" name="HDL-32E">
+  <xacro:macro name="HDL-32E" params="parent name *origin">
     <joint name="${name}_base_mount_joint" type="fixed">
       <xacro:insert_block name="origin" />
@@ -18,24 +18,16 @@
         </material>
         <geometry>
-          <mesh filename="package://velodyne_description/meshes/VLP16_base_1.stl" />
-        </geometry>
-      </visual>
-      <visual>
-        <material name="lightgrey" >
-          <color rgba="0.5 0.5 0.5 1"/>
-        </material>
-        <geometry>
-          <mesh filename="package://velodyne_description/meshes/VLP16_base_2.stl" />
+          <mesh filename="package://velodyne_description/meshes/HDL32E_base.stl" />
         </geometry>
       </visual>
       <collision>
-        <origin rpy="0 0 0" xyz="0 0 0.03585"/>
+        <origin rpy="0 0 0" xyz="0 0 0.07212"/>
         <geometry>
-          <cylinder radius="0.0516" length="0.0717"/>
+          <cylinder radius="0.04267" length="0.14424"/>
         </geometry>
       </collision>
     </link>
     <joint name="${name}_base_scan_joint" type="fixed" >
-      <origin xyz="0 0 0.0377" rpy="0 0 0" />
+      <origin xyz="0 0 0.09081" rpy="0 0 0" />
       <parent link="${name}_base_link" />
       <child link="${name}"/>
@@ -48,10 +40,10 @@
       </inertial>
       <visual>
-        <material name="black" >
-          <color rgba=".1 .1 .1 1"/>
+        <material name="lightgrey" >
+          <color rgba="0.5 0.5 0.5 1"/>
         </material>
-        <origin xyz="0 0 -0.0377" />
+        <origin xyz="0 0 -0.09081" rpy="0 0 0" />
         <geometry>
-          <mesh filename="package://velodyne_description/meshes/VLP16_scan.stl" />
+          <mesh filename="package://velodyne_description/meshes/HDL32E_scan.stl" />
         </geometry>
       </visual>
@@ -59,5 +51,5 @@
     <!-- Gazebo requires the velodyne_gazebo_plugins package -->
     <gazebo reference="${name}">
-      <sensor type="ray" name="${name}-VLP16">
+      <sensor type="ray" name="${name}-HDL32E">
         <pose>0 0 0 0 0 0</pose>
         <visualize>false</visualize>
@@ -66,5 +58,5 @@
           <scan>
             <horizontal>
-              <samples>1875</samples>
+              <samples>2187</samples>
               <resolution>1</resolution>
               <min_angle>-${M_PI}</min_angle>
@@ -72,8 +64,8 @@
             </horizontal>
             <vertical>
-              <samples>16</samples>
+              <samples>32</samples>
               <resolution>1</resolution>
-              <min_angle>-${15.0*M_PI/180.0}</min_angle>
-              <max_angle> ${15.0*M_PI/180.0}</max_angle>
+              <min_angle>-${10.67*M_PI/180.0}</min_angle> <!-- This is backwards to support gazebo 2 -->
+              <max_angle> ${30.67*M_PI/180.0}</max_angle>
             </vertical>
           </scan>
@@ -102,5 +94,5 @@
     </gazebo>
     <gazebo reference="${name}">
-      <material>Gazebo/Black</material>
+      <material>Gazebo/Grey</material>
     </gazebo>
   </xacro:macro>

Commit message: Changed to DAE meshes

File: velodyne_description/urdf/HDL-32E.urdf.xacro (robot description, xacro)
@@ -2,4 +2,7 @@
 <robot xmlns:xacro="http://ros.org/wiki/xacro" name="HDL-32E">
   <xacro:macro name="HDL-32E" params="parent name *origin">
+    <material name="hdl_lightgrey">
+      <color rgba="0.55 0.55 0.55 1"/>
+    </material>
     <joint name="${name}_base_mount_joint" type="fixed">
       <xacro:insert_block name="origin" />
@@ -14,10 +17,8 @@
       </inertial>
       <visual>
-        <material name="lightgrey" >
-          <color rgba="0.5 0.5 0.5 1"/>
-        </material>
         <geometry>
-          <mesh filename="package://velodyne_description/meshes/HDL32E_base.stl" />
+          <mesh filename="package://velodyne_description/meshes/HDL32E_base.dae" />
         </geometry>
+        <material name="hdl_lightgrey"/>
       </visual>
       <collision>
@@ -40,11 +41,9 @@
       </inertial>
       <visual>
-        <material name="lightgrey" >
-          <color rgba="0.5 0.5 0.5 1"/>
-        </material>
         <origin xyz="0 0 -0.09081" rpy="0 0 0" />
         <geometry>
-          <mesh filename="package://velodyne_description/meshes/HDL32E_scan.stl" />
+          <mesh filename="package://velodyne_description/meshes/HDL32E_scan.dae" />
         </geometry>
+        <material name="hdl_lightgrey"/>
       </visual>
     </link>
@@ -90,10 +89,4 @@
       </sensor>
     </gazebo>
-    <gazebo reference="${name}_base_link">
-      <material>Gazebo/Grey</material>
-    </gazebo>
-    <gazebo reference="${name}">
-      <material>Gazebo/Grey</material>
-    </gazebo>
   </xacro:macro>
 </robot>

File: velodyne_description/urdf/VLP-16.urdf.xacro (robot description, xacro)
@@ -2,4 +2,10 @@
 <robot xmlns:xacro="http://ros.org/wiki/xacro" name="VLP-16">
   <xacro:macro name="VLP-16" params="parent name *origin">
+    <material name="vlp_lightgrey">
+      <color rgba="0.55 0.55 0.55 1"/>
+    </material>
+    <material name="vlp_black">
+      <color rgba="0.1 0.1 0.1 1"/>
+    </material>
     <joint name="${name}_base_mount_joint" type="fixed">
       <xacro:insert_block name="origin" />
@@ -14,18 +20,14 @@
       </inertial>
       <visual>
-        <material name="lightgrey" >
-          <color rgba="0.5 0.5 0.5 1"/>
-        </material>
         <geometry>
-          <mesh filename="package://velodyne_description/meshes/VLP16_base_1.stl" />
+          <mesh filename="package://velodyne_description/meshes/VLP16_base_1.dae" />
         </geometry>
+        <material name="vlp_lightgrey"/>
       </visual>
       <visual>
-        <material name="lightgrey" >
-          <color rgba="0.5 0.5 0.5 1"/>
-        </material>
         <geometry>
-          <mesh filename="package://velodyne_description/meshes/VLP16_base_2.stl" />
+          <mesh filename="package://velodyne_description/meshes/VLP16_base_2.dae" />
         </geometry>
+        <material name="vlp_lightgrey"/>
       </visual>
       <collision>
@@ -48,11 +50,9 @@
       </inertial>
       <visual>
-        <material name="black" >
-          <color rgba=".1 .1 .1 1"/>
-        </material>
         <origin xyz="0 0 -0.0377" />
         <geometry>
-          <mesh filename="package://velodyne_description/meshes/VLP16_scan.stl" />
+          <mesh filename="package://velodyne_description/meshes/VLP16_scan.dae" />
         </geometry>
+        <material name="vlp_black"/>
       </visual>
     </link>
@@ -98,10 +98,4 @@
       </sensor>
     </gazebo>
-    <gazebo reference="${name}_base_link">
-      <material>Gazebo/Grey</material>
-    </gazebo>
-    <gazebo reference="${name}">
-      <material>Gazebo/Black</material>
-    </gazebo>
   </xacro:macro>
 </robot>

Commit message: Added example urdf and gazebo

File: velodyne_description/urdf/HDL-32E.urdf.xacro (robot description, xacro)
@@ -1,5 +1,6 @@
 <?xml version="1.0"?>
 <robot xmlns:xacro="http://ros.org/wiki/xacro" name="HDL-32E">
-  <xacro:macro name="HDL-32E" params="parent name *origin">
+  <xacro:macro name="HDL-32E" params="parent name topic *origin">
+    <xacro:property name="M_PI" value="3.1415926535897931" />
     <material name="hdl_lightgrey">
       <color rgba="0.55 0.55 0.55 1"/>
@@ -81,5 +82,5 @@
         </ray>
         <plugin name="gazebo_ros_laser_controller" filename="libgazebo_ros_velodyne_laser.so">
-          <topicName>/${name}/points</topicName>
+          <topicName>${topic}</topicName>
           <frameName>/${name}</frameName>
           <min_range>0.9</min_range>

File: velodyne_description/urdf/VLP-16.urdf.xacro (robot description, xacro)
@@ -1,5 +1,6 @@
 <?xml version="1.0"?>
 <robot xmlns:xacro="http://ros.org/wiki/xacro" name="VLP-16">
-  <xacro:macro name="VLP-16" params="parent name *origin">
+  <xacro:macro name="VLP-16" params="parent name topic *origin">
+    <xacro:property name="M_PI" value="3.1415926535897931" />
     <material name="vlp_lightgrey">
       <color rgba="0.55 0.55 0.55 1"/>
@@ -90,5 +91,5 @@
         </ray>
         <plugin name="gazebo_ros_laser_controller" filename="libgazebo_ros_velodyne_laser.so">
-          <topicName>/${name}/points</topicName>
+          <topicName>${topic}</topicName>
           <frameName>/${name}</frameName>
           <min_range>0.9</min_range>

Commit message: Materials caused problems with more than one sensors. Removed.

File: velodyne_description/urdf/HDL-32E.urdf.xacro (robot description, xacro)
@@ -1,9 +1,6 @@
 <?xml version="1.0"?>
-<robot xmlns:xacro="http://ros.org/wiki/xacro" name="HDL-32E">
+<robot xmlns:xacro="http://www.ros.org/wiki/xacro" name="HDL-32E">
   <xacro:macro name="HDL-32E" params="parent name topic *origin">
     <xacro:property name="M_PI" value="3.1415926535897931" />
-    <material name="hdl_lightgrey">
-      <color rgba="0.55 0.55 0.55 1"/>
-    </material>
     <joint name="${name}_base_mount_joint" type="fixed">
       <xacro:insert_block name="origin" />
@@ -21,5 +18,4 @@
           <mesh filename="package://velodyne_description/meshes/HDL32E_base.dae" />
         </geometry>
-        <material name="hdl_lightgrey"/>
       </visual>
       <collision>
@@ -46,5 +42,4 @@
           <mesh filename="package://velodyne_description/meshes/HDL32E_scan.dae" />
         </geometry>
-        <material name="hdl_lightgrey"/>
       </visual>
     </link>

File: velodyne_description/urdf/VLP-16.urdf.xacro (robot description, xacro)
@@ -1,12 +1,6 @@
 <?xml version="1.0"?>
-<robot xmlns:xacro="http://ros.org/wiki/xacro" name="VLP-16">
+<robot xmlns:xacro="http://www.ros.org/wiki/xacro" name="VLP-16">
   <xacro:macro name="VLP-16" params="parent name topic *origin">
     <xacro:property name="M_PI" value="3.1415926535897931" />
-    <material name="vlp_lightgrey">
-      <color rgba="0.55 0.55 0.55 1"/>
-    </material>
-    <material name="vlp_black">
-      <color rgba="0.1 0.1 0.1 1"/>
-    </material>
     <joint name="${name}_base_mount_joint" type="fixed">
       <xacro:insert_block name="origin" />
@@ -24,5 +18,4 @@
           <mesh filename="package://velodyne_description/meshes/VLP16_base_1.dae" />
         </geometry>
-        <material name="vlp_lightgrey"/>
       </visual>
       <visual>
@@ -30,5 +23,4 @@
           <mesh filename="package://velodyne_description/meshes/VLP16_base_2.dae" />
         </geometry>
-        <material name="vlp_lightgrey"/>
       </visual>
       <collision>
@@ -55,5 +47,4 @@
           <mesh filename="package://velodyne_description/meshes/VLP16_scan.dae" />
         </geometry>
-        <material name="vlp_black"/>
       </visual>
     </link>

File: velodyne_description/urdf/example.urdf.xacro (robot description, xacro)
@@ -1,4 +1,4 @@
 <?xml version="1.0"?>
-<robot xmlns:xacro="http://ros.org/wiki/xacro" name="example">
+<robot xmlns:xacro="http://www.ros.org/wiki/xacro" name="example">
   <!-- Base Footprint -->
   <link name="base_footprint" />

Commit message: Moved M_PI property out of macro to support multiple instances

File: velodyne_description/urdf/HDL-32E.urdf.xacro (robot description, xacro)
@@ -1,6 +1,6 @@
 <?xml version="1.0"?>
 <robot xmlns:xacro="http://www.ros.org/wiki/xacro" name="HDL-32E">
+  <xacro:property name="M_PI" value="3.1415926535897931" />
   <xacro:macro name="HDL-32E" params="parent name topic *origin">
-    <xacro:property name="M_PI" value="3.1415926535897931" />
     <joint name="${name}_base_mount_joint" type="fixed">
       <xacro:insert_block name="origin" />

File: velodyne_description/urdf/VLP-16.urdf.xacro (robot description, xacro)
@@ -1,6 +1,6 @@
 <?xml version="1.0"?>
 <robot xmlns:xacro="http://www.ros.org/wiki/xacro" name="VLP-16">
+  <xacro:property name="M_PI" value="3.1415926535897931" />
   <xacro:macro name="VLP-16" params="parent name topic *origin">
-    <xacro:property name="M_PI" value="3.1415926535897931" />
     <joint name="${name}_base_mount_joint" type="fixed">
       <xacro:insert_block name="origin" />

Commit message: Added many URDF parameters, and set example sample count to reasonable values

File: velodyne_description/urdf/HDL-32E.urdf.xacro (robot description, xacro)
@@ -2,5 +2,5 @@
 <robot xmlns:xacro="http://www.ros.org/wiki/xacro" name="HDL-32E">
   <xacro:property name="M_PI" value="3.1415926535897931" />
-  <xacro:macro name="HDL-32E" params="parent name topic *origin">
+  <xacro:macro name="HDL-32E" params="*origin parent:=base_link name:=velodyne topic:=/velodyne_points hz:=10 lasers:=32 samples:=2187 min_range:=0.9 max_range:=130.0 noise:=0.008 min_angle:=-${M_PI} max_angle:=${M_PI}">
     <joint name="${name}_base_mount_joint" type="fixed">
       <xacro:insert_block name="origin" />
@@ -49,15 +49,15 @@
         <pose>0 0 0 0 0 0</pose>
         <visualize>false</visualize>
-        <update_rate>10</update_rate>
+        <update_rate>${hz}</update_rate>
         <ray>
           <scan>
             <horizontal>
-              <samples>2187</samples> <!-- Change this to 500 if gazebo keeps timing out -->
+              <samples>${samples}</samples>
               <resolution>1</resolution>
-              <min_angle>-${M_PI}</min_angle>
-              <max_angle> ${M_PI}</max_angle>
+              <min_angle>${min_angle}</min_angle>
+              <max_angle>${max_angle}</max_angle>
             </horizontal>
             <vertical>
-              <samples>32</samples>
+              <samples>${lasers}</samples>
               <resolution>1</resolution>
               <min_angle>-${30.67*M_PI/180.0}</min_angle>
@@ -79,7 +79,7 @@
           <topicName>${topic}</topicName>
           <frameName>/${name}</frameName>
-          <min_range>0.9</min_range>
-          <max_range>130.0</max_range>
-          <gaussianNoise>0.008</gaussianNoise>
+          <min_range>${min_range}</min_range>
+          <max_range>${max_range}</max_range>
+          <gaussianNoise>${noise}</gaussianNoise>
         </plugin>
       </sensor>

Commit message: Increased minimum collision range to prevent self-clipping when in motion

File: velodyne_description/urdf/HDL-32E.urdf.xacro (robot description, xacro)
@@ -2,5 +2,5 @@
 <robot xmlns:xacro="http://www.ros.org/wiki/xacro" name="HDL-32E">
   <xacro:property name="M_PI" value="3.1415926535897931" />
-  <xacro:macro name="HDL-32E" params="*origin parent:=base_link name:=velodyne topic:=/velodyne_points hz:=10 lasers:=32 samples:=2187 min_range:=0.9 max_range:=130.0 noise:=0.008 min_angle:=-${M_PI} max_angle:=${M_PI}">
+  <xacro:macro name="HDL-32E" params="*origin parent:=base_link name:=velodyne topic:=/velodyne_points hz:=10 lasers:=32 samples:=2187 collision_range:=0.3 min_range:=0.9 max_range:=130.0 noise:=0.008 min_angle:=-${M_PI} max_angle:=${M_PI}">
     <joint name="${name}_base_mount_joint" type="fixed">
       <xacro:insert_block name="origin" />
@@ -66,6 +66,6 @@
           </scan>
           <range>
-            <min>0.055</min>
-            <max>140.0</max>
+            <min>${collision_range}</min>
+            <max>${max_range+1}</max>
             <resolution>0.001</resolution>
           </range>

Commit message: Merged in xqms/velodyne_simulator/inertia (pull request #3)
velodyne_description: more realistic inertia tensor for VLP-16

* velodyne_description: more realistic inertia tensor for VLP-16

* velodyne_description: VLP-16: fix whitespace

* velodyne_description: inertia tensor for HDL-32E

File: velodyne_description/urdf/HDL-32E.urdf.xacro (robot description, xacro)
@@ -10,7 +10,9 @@
     <link name="${name}_base_link">
       <inertial>
-        <mass value="0.1"/>
-        <origin xyz="0 0 0"/>
-        <inertia ixx="0.1" ixy="0" ixz="0" iyy="0.1" iyz="0" izz="0.1"/>
+        <mass value="1.0"/>
+        <origin xyz="0 0 0.07212"/>
+        <inertia ixx="${(1.0 * (3.0*0.04267*0.04267 + 0.14424*0.14424)) / 12.0}" ixy="0" ixz="0"
+          iyy="${(1.0 * (3.0*0.04267*0.04267 + 0.14424*0.14424)) / 12.0}" iyz="0"
+          izz="${0.5 * 1.0 * (0.04267*0.04267)}"/>
       </inertial>
       <visual>
@@ -33,7 +35,7 @@
     <link name="${name}">
       <inertial>
-        <mass value="0.1"/>
+        <mass value="0.01"/>
         <origin xyz="0 0 0"/>
-        <inertia ixx="0.1" ixy="0" ixz="0" iyy="0.1" iyz="0" izz="0.1"/>
+        <inertia ixx="1e-7" ixy="0" ixz="0" iyy="1e-7" iyz="0" izz="1e-7"/>
       </inertial>
       <visual>

File: velodyne_description/urdf/VLP-16.urdf.xacro (robot description, xacro)
@@ -10,7 +10,9 @@
     <link name="${name}_base_link">
       <inertial>
-        <mass value="0.1"/>
-        <origin xyz="0 0 0"/>
-        <inertia ixx="0.1" ixy="0" ixz="0" iyy="0.1" iyz="0" izz="0.1"/>
+        <mass value="0.83"/>
+        <origin xyz="0 0 0.03585"/>
+        <inertia ixx="${(0.83 * (3.0*0.0516*0.0516 + 0.0717*0.0717)) / 12.0}" ixy="0" ixz="0"
+          iyy="${(0.83 * (3.0*0.0516*0.0516 + 0.0717*0.0717)) / 12.0}" iyz="0"
+          izz="${0.5 * 0.83 * (0.0516*0.0516)}"/>
       </inertial>
       <visual>
@@ -38,7 +40,7 @@
     <link name="${name}">
       <inertial>
-        <mass value="0.1"/>
+        <mass value="0.01"/>
         <origin xyz="0 0 0"/>
-        <inertia ixx="0.1" ixy="0" ixz="0" iyy="0.1" iyz="0" izz="0.1"/>
+        <inertia ixx="1e-7" ixy="0" ixz="0" iyy="1e-7" iyz="0" izz="1e-7"/>
       </inertial>
       <visual>
