Commit message: Updated urdf syntax for jade

File: velodyne_description/urdf/VLP-16.urdf.xacro (robot description, xacro)
@@ -1,7 +1,7 @@
 <?xml version="1.0"?>
-<robot name="sensor_vlp16" xmlns:xacro="http://ros.org/wiki/xacro">
-  <macro name="VLP-16" params="parent name *origin">
+<robot xmlns:xacro="http://ros.org/wiki/xacro" name="VLP-16">
+  <xacro:macro name="VLP-16" params="parent name *origin">
     <joint name="${name}_base_mount_joint" type="fixed">
-      <insert_block name="origin" />
+      <xacro:insert_block name="origin" />
       <parent link="${parent}"/>
       <child link="${name}_base_link"/>
@@ -97,4 +97,4 @@
       <material>Gazebo/Black</material>
     </gazebo>
-  </macro>
+  </xacro:macro>
 </robot>

Commit message: Reduce VLP16 sensor mass and inertia

File: velodyne_description/urdf/VLP-16.urdf.xacro (robot description, xacro)
@@ -10,9 +10,7 @@
     <link name="${name}_base_link">
       <inertial>
-        <mass value="0.83"/>
+        <mass value="0.01"/>
         <origin xyz="0 0 0.03585"/>
-        <inertia ixx="${(0.83 * (3.0*0.0516*0.0516 + 0.0717*0.0717)) / 12.0}" ixy="0" ixz="0"
-          iyy="${(0.83 * (3.0*0.0516*0.0516 + 0.0717*0.0717)) / 12.0}" iyz="0"
-          izz="${0.5 * 0.83 * (0.0516*0.0516)}"/>
+        <inertia ixx="1e-7" ixy="0" ixz="0" iyy="1e-7" iyz="0" izz="1e-7"/>
       </inertial>
       <visual>

Commit message: [velodyne-simulator] Revert changes to subtree
(cherry picked from commit 18d7ec6a753d74f803b07cca25e5517bfa2e8155)

File: velodyne_description/urdf/VLP-16.urdf.xacro (robot description, xacro)
@@ -10,7 +10,9 @@
     <link name="${name}_base_link">
       <inertial>
-        <mass value="0.01"/>
+        <mass value="0.83"/>
         <origin xyz="0 0 0.03585"/>
-        <inertia ixx="1e-7" ixy="0" ixz="0" iyy="1e-7" iyz="0" izz="1e-7"/>
+        <inertia ixx="${(0.83 * (3.0*0.0516*0.0516 + 0.0717*0.0717)) / 12.0}" ixy="0" ixz="0"
+          iyy="${(0.83 * (3.0*0.0516*0.0516 + 0.0717*0.0717)) / 12.0}" iyz="0"
+          izz="${0.5 * 0.83 * (0.0516*0.0516)}"/>
       </inertial>
       <visual>
