Commit message: Change frame for the rotating link

File: velodyne_description/urdf/VU-8.urdf-rotating.xacro (robot description, xacro)
@@ -40,5 +40,5 @@
       </collision>
     </link>
-    <link name="${name}">
+    <link name="rotating_${name}">
       <inertial>
         <mass value="1e-2"/>
@@ -56,5 +56,5 @@
       <origin xyz="0 0 0.0377" rpy="0 0 0" />
       <parent link="${name}_base_link" />
-      <child link="${name}"/>
+      <child link="rotating_${name}"/>
       <limit effort="1000.0" lower="-0.5" upper="0.5" velocity="0.5"/>
       <axis xyz="0 0 1" />
@@ -70,5 +70,5 @@
     </transmission>
     <!-- Gazebo requires the velodyne_gazebo_plugins package -->
-    <gazebo reference="${name}">
+    <gazebo reference="rotating_${name}">
       <xacro:if value="${gpu}">
         <sensor type="gpu_ray" name="${name}-VU8">
@@ -104,5 +104,5 @@
           <plugin name="gazebo_ros_laser_controller" filename="libgazebo_ros_velodyne_gpu_laser.so">
             <topicName>${topic}</topicName>
-            <frameName>${name}</frameName>
+            <frameName>rotating_${name}</frameName>
             <min_range>${min_range}</min_range>
             <max_range>${max_range}</max_range>
@@ -144,5 +144,5 @@
           <plugin name="gazebo_ros_laser_controller" filename="libgazebo_ros_velodyne_laser.so">
             <topicName>${topic}</topicName>
-            <frameName>${name}</frameName>
+            <frameName>rotating_${name}</frameName>
             <min_range>${min_range}</min_range>
             <max_range>${max_range}</max_range>

Commit message: Add supoort for rotating velodyne in GazeboRosVelodyneLaser

File: velodyne_description/urdf/VU-8.urdf-rotating.xacro (robot description, xacro)
@@ -57,5 +57,5 @@
       <parent link="${name}_base_link" />
       <child link="rotating_${name}"/>
-      <limit effort="1000.0" lower="-0.5" upper="0.5" velocity="0.5"/>
+      <limit effort="10.0" lower="-0.5" upper="0.5" velocity="0.1"/>
       <axis xyz="0 0 1" />
     </joint>
@@ -108,4 +108,6 @@
             <max_range>${max_range}</max_range>
             <gaussianNoise>${noise}</gaussianNoise>
+            <staticFrameName>${name}_base_link</staticFrameName>
+            <staticTopicName>${topic}_static</staticTopicName>
           </plugin>
         </sensor>
@@ -148,4 +150,6 @@
             <max_range>${max_range}</max_range>
             <gaussianNoise>${noise}</gaussianNoise>
+            <staticFrameName>${name}_base_link</staticFrameName>
+            <staticTopicName>${topic}_static</staticTopicName>
           </plugin>
         </sensor>

Commit message: [VU-8] Move angles to parameters

File: velodyne_description/urdf/VU-8.urdf-rotating.xacro (robot description, xacro)
@@ -2,14 +2,21 @@
 <robot xmlns:xacro="http://www.ros.org/wiki/xacro" name="VU-8">
   <xacro:property name="M_PI" value="3.1415926535897931" />
-  <!-- Minimum horizontal angle is -100 DEG - Wide FOV -->
-  <xacro:property name="min_horizontal_angle" value="-3.14159" />
-  <!-- Maximum horizontal angle is 100 DEG - Wide FOV -->
-  <xacro:property name="max_horizontal_angle" value="3.14159" />
-  <!-- Minimum vertical angle is -3 DEG -->
-  <xacro:property name="min_vertical_angle" value="-0.523599" />
-  <!-- Maximum vertical angle is 3 DEG-->
-  <xacro:property name="max_vertical_angle" value="0.523599" />
   <xacro:macro name="VU-8" params="
-    *origin parent:=base_link name:=leddar topic:=/leddar_points hz:=10 lasers:=8 samples:=1875 collision_range:=0.3 min_range:=0.1 max_range:=130.0 noise:=0.008 gpu:=false">
+    *origin
+    parent:=base_link
+    name:=leddar
+    topic:=/lidar_points
+    hz:=10
+    lasers:=8
+    samples:=1875
+    collision_range:=0.3
+    min_range:=0.1
+    max_range:=130.0
+    noise:=0.008
+    min_horizontal_angle:=-3.14159
+    max_horizontal_angle:=3.14159
+    min_vertical_angle:=-0.523599
+    max_vertical_angle:=0.523599
+    gpu:=false">
     <joint name="${name}_base_mount_joint" type="fixed">
       <xacro:insert_block name="origin" />

File: velodyne_description/urdf/VU-8.urdf.xacro (robot description, xacro)
@@ -2,14 +2,21 @@
 <robot xmlns:xacro="http://www.ros.org/wiki/xacro" name="VU-8">
   <xacro:property name="M_PI" value="3.1415926535897931" />
-  <!-- Minimum horizontal angle is -100 DEG - Wide FOV -->
-  <xacro:property name="min_horizontal_angle" value="-3.14159" />
-  <!-- Maximum horizontal angle is 100 DEG - Wide FOV -->
-  <xacro:property name="max_horizontal_angle" value="3.14159" />
-  <!-- Minimum vertical angle is -3 DEG -->
-  <xacro:property name="min_vertical_angle" value="-0.523599" />
-  <!-- Maximum vertical angle is 3 DEG-->
-  <xacro:property name="max_vertical_angle" value="0.523599" />
   <xacro:macro name="VU-8" params="
-    *origin parent:=base_link name:=leddar topic:=/leddar_points hz:=10 lasers:=8 samples:=1875 collision_range:=0.3 min_range:=0.1 max_range:=130.0 noise:=0.008 gpu:=false">
+    *origin
+    parent:=base_link
+    name:=leddar
+    topic:=/lidar_points
+    hz:=10
+    lasers:=8
+    samples:=1875
+    collision_range:=0.3
+    min_range:=0.1
+    max_range:=130.0
+    noise:=0.008
+    min_horizontal_angle:=-3.14159
+    max_horizontal_angle:=3.14159
+    min_vertical_angle:=-0.523599
+    max_vertical_angle:=0.523599
+    gpu:=false">
     <joint name="${name}_base_mount_joint" type="fixed">
       <xacro:insert_block name="origin" />
