Commit message: [LiDAR-X] Rename plugin to lidar-x

File: velodyne_description/urdf/LiDAR-X-rotating.urdf.xacro (robot description, xacro)
@@ -2,5 +2,5 @@
 <robot xmlns:xacro="http://www.ros.org/wiki/xacro" name="VU-8">
   <xacro:property name="M_PI" value="3.1415926535897931" />
-  <xacro:macro name="VU-8" params="
+  <xacro:macro name="lidar-x" params="
     *origin
     parent:=base_link

File: velodyne_description/urdf/LiDAR-X.urdf.xacro (robot description, xacro)
@@ -2,5 +2,5 @@
 <robot xmlns:xacro="http://www.ros.org/wiki/xacro" name="VU-8">
   <xacro:property name="M_PI" value="3.1415926535897931" />
-  <xacro:macro name="VU-8" params="
+  <xacro:macro name="lidar-x" params="
     *origin
     parent:=base_link
